File: oscilloscope-probing/lab/boards/prbs-generator/leds.kicad_sch (KiCad schematic)
At the start: 42 parts, among them U3 SX1502_QFN20, U4 SX1502_QFN20

Commit message: Continued work on PRBS board layout
Connections:
- net at D2.1 (K): now also U3.16 (IO_5); no longer U3.9 (IO_2)
- net at D9.1 (K): now also U3.19 (IO_6); no longer U3.6 (IO_1)
- net at U3.15 (IO_4): now also D1.1 (K); no longer D3.1 (K)
- net at D11.1 (K): now also U3.6 (IO_1); no longer U3.16 (IO_5)
- net at D4.1 (K): now also U3.9 (IO_2); no longer U3.19 (IO_6)
- net at U3.20 (IO_7): now also D10.1 (K); no longer D12.1 (K)
- net at U3.5 (IO_0): now also D3.1 (K); no longer D1.1 (K)
- net at U3.10 (IO_3): now also D12.1 (K); no longer D10.1 (K)
Other:
- moved on the sheet: D2, D9, R12, R5, U3B, U3C
Changed lines of the file:
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@@
   (title_block
     (title "PRBS Generator")
-    (date "2022-03-18")
+    (date "2022-03-19")
     (rev "0.1")
     (company "Antikernel Labs")
@@
   (junction (at 177.8 28.575) (diameter 0) (color 0 0 0 0)
   )
+  (junction (at 177.8 26.035) (diameter 0) (color 0 0 0 0)
+  )
   (junction (at 177.8 106.68) (diameter 0) (color 0 0 0 0)
   )
@@
   )
   (junction (at 53.34 37.465) (diameter 0) (color 0 0 0 0)
-  )
-  (junction (at 177.8 26.035) (diameter 0) (color 0 0 0 0)
   )
   (junction (at 40.005 90.805) (diameter 0) (color 0 0 0 0)
@@
     (stroke (width 0) (type default) (color 0 0 0 0))
   )
-  (wire (pts (xy 177.8 28.575) (xy 177.8 26.035))
+  (wire (pts (xy 177.8 23.495) (xy 177.8 26.035))
     (stroke (width 0) (type default) (color 0 0 0 0))
   )
@@
     (stroke (width 0) (type default) (color 0 0 0 0))
   )
-  (wire (pts (xy 177.8 26.035) (xy 177.8 23.495))
-    (stroke (width 0) (type default) (color 0 0 0 0))
-  )
   (wire (pts (xy 92.71 30.48) (xy 92.71 33.02))
     (stroke (width 0) (type default) (color 0 0 0 0))
@@
   )
   (wire (pts (xy 138.43 23.495) (xy 143.51 23.495))
+    (stroke (width 0) (type default) (color 0 0 0 0))
+  )
+  (wire (pts (xy 177.8 26.035) (xy 177.8 28.575))
     (stroke (width 0) (type default) (color 0 0 0 0))
   )
@@
     (pin "2")
   )
-  (symbol (lib_id "device:LED") (at 147.32 28.575 0) (unit 1)
-    (in_bom yes) (on_board yes)
-    (property "Reference" "D2" (id 0) (at 146.685 32.385 0))
-    (property "Value" "GREEN" (id 1) (at 146.685 34.29 0))
-    (property "Footprint" "azonenberg_pcb:EIA_0805_LED" (id 2) (at 147.32 28.575 0)
-      (effects (font (size 1.27 1.27)) hide)
-    )
-    (property "Datasheet" "" (id 3) (at 147.32 28.575 0)
+  (symbol (lib_id "device:LED") (at 166.37 26.035 0) (unit 1)
+    (in_bom yes) (on_board yes)
+    (property "Reference" "D2" (id 0) (at 165.735 29.845 0))
+    (property "Value" "GREEN" (id 1) (at 165.735 31.75 0))
+    (property "Footprint" "azonenberg_pcb:EIA_0805_LED" (id 2) (at 166.37 26.035 0)
+      (effects (font (size 1.27 1.27)) hide)
+    )
+    (property "Datasheet" "" (id 3) (at 166.37 26.035 0)
       (effects (font (size 1.27 1.27)) hide)
     )
@@
     (pin "2")
   )
-  (symbol (lib_id "device:LED") (at 166.37 26.035 0) (unit 1)
-    (in_bom yes) (on_board yes)
-    (property "Reference" "D9" (id 0) (at 167.005 20.32 0))
-    (property "Value" "GREEN" (id 1) (at 166.37 22.225 0))
-    (property "Footprint" "azonenberg_pcb:EIA_0805_LED" (id 2) (at 166.37 26.035 0)
-      (effects (font (size 1.27 1.27)) hide)
-    )
-    (property "Datasheet" "" (id 3) (at 166.37 26.035 0)
+  (symbol (lib_id "device:LED") (at 147.32 28.575 0) (unit 1)
+    (in_bom yes) (on_board yes)
+    (property "Reference" "D9" (id 0) (at 147.955 22.86 0))
+    (property "Value" "GREEN" (id 1) (at 147.32 24.765 0))
+    (property "Footprint" "azonenberg_pcb:EIA_0805_LED" (id 2) (at 147.32 28.575 0)
+      (effects (font (size 1.27 1.27)) hide)
+    )
+    (property "Datasheet" "" (id 3) (at 147.32 28.575 0)
       (effects (font (size 1.27 1.27)) hide)
     )
@@
     (pin "2")
   )
-  (symbol (lib_id "special-azonenberg:SX1502_QFN20") (at 135.89 59.69 0) (mirror y) (unit 3)
-    (in_bom yes) (on_board yes)
-    (property "Reference" "U3" (id 0) (at 132.08 45.6143 0))
-    (property "Value" "SX1502_QFN20" (id 1) (at 132.08 48.3894 0))
-    (property "Footprint" "azonenberg_pcb:QFN_20_0.4MM_3x3MM" (id 2) (at 135.89 59.69 0)
-      (effects (font (size 1.27 1.27)) hide)
-    )
-    (property "Datasheet" "" (id 3) (at 135.89 59.69 0)
+  (symbol (lib_id "special-azonenberg:SX1502_QFN20") (at 135.89 32.385 0) (mirror y) (unit 3)
+    (in_bom yes) (on_board yes)
+    (property "Reference" "U3" (id 0) (at 132.08 18.3093 0))
+    (property "Value" "SX1502_QFN20" (id 1) (at 132.08 21.0844 0))
+    (property "Footprint" "azonenberg_pcb:QFN_20_0.4MM_3x3MM" (id 2) (at 135.89 32.385 0)
+      (effects (font (size 1.27 1.27)) hide)
+    )
+    (property "Datasheet" "" (id 3) (at 135.89 32.385 0)
       (effects (font (size 1.27 1.27)) hide)
     )
@@
     (pin "2")
   )
-  (symbol (lib_id "device:R") (at 173.99 26.035 90) (unit 1)
-    (in_bom yes) (on_board yes)
-    (property "Reference" "R12" (id 0) (at 180.34 26.035 90))
-    (property "Value" "470" (id 1) (at 173.99 26.035 90))
-    (property "Footprint" "azonenberg_pcb:EIA_0402_RES_NOSILK" (id 2) (at 173.99 27.813 90)
-      (effects (font (size 1.27 1.27)) hide)
-    )
-    (property "Datasheet" "" (id 3) (at 173.99 26.035 0)
+  (symbol (lib_id "device:R") (at 154.94 28.575 90) (unit 1)
+    (in_bom yes) (on_board yes)
+    (property "Reference" "R12" (id 0) (at 161.29 28.575 90))
+    (property "Value" "470" (id 1) (at 154.94 28.575 90))
+    (property "Footprint" "azonenberg_pcb:EIA_0402_RES_NOSILK" (id 2) (at 154.94 30.353 90)
+      (effects (font (size 1.27 1.27)) hide)
+    )
+    (property "Datasheet" "" (id 3) (at 154.94 28.575 0)
       (effects (font (size 1.27 1.27)) hide)
     )
@@
     (pin "2")
   )
-  (symbol (lib_id "special-azonenberg:SX1502_QFN20") (at 135.89 32.385 0) (mirror y) (unit 2)
-    (in_bom yes) (on_board yes) (fields_autoplaced)
-    (property "Reference" "U3" (id 0) (at 132.08 18.3093 0))
-    (property "Value" "SX1502_QFN20" (id 1) (at 132.08 21.0844 0))
-    (property "Footprint" "azonenberg_pcb:QFN_20_0.4MM_3x3MM" (id 2) (at 135.89 32.385 0)
-      (effects (font (size 1.27 1.27)) hide)
-    )
-    (property "Datasheet" "" (id 3) (at 135.89 32.385 0)
+  (symbol (lib_id "special-azonenberg:SX1502_QFN20") (at 135.89 59.69 0) (mirror y) (unit 2)
+    (in_bom yes) (on_board yes)
+    (property "Reference" "U3" (id 0) (at 132.08 45.6143 0))
+    (property "Value" "SX1502_QFN20" (id 1) (at 132.08 48.3894 0))
+    (property "Footprint" "azonenberg_pcb:QFN_20_0.4MM_3x3MM" (id 2) (at 135.89 59.69 0)
+      (effects (font (size 1.27 1.27)) hide)
+    )
+    (property "Datasheet" "" (id 3) (at 135.89 59.69 0)
       (effects (font (size 1.27 1.27)) hide)
     )
@@
     (pin "2")
   )
-  (symbol (lib_id "device:R") (at 154.94 28.575 90) (unit 1)
-    (in_bom yes) (on_board yes)
-    (property "Reference" "R5" (id 0) (at 158.75 27.305 90))
-    (property "Value" "470" (id 1) (at 154.94 28.575 90))
-    (property "Footprint" "azonenberg_pcb:EIA_0402_RES_NOSILK" (id 2) (at 154.94 30.353 90)
-      (effects (font (size 1.27 1.27)) hide)
-    )
-    (property "Datasheet" "" (id 3) (at 154.94 28.575 0)
-      (effects (font (size 1.27 1.27)) hide)
-    )
+  (symbol (lib_id "device:R") (at 173.99 26.035 90) (unit 1)
+    (in_bom yes) (on_board yes)
+    (property "Reference" "R5" (id 0) (at 177.8 24.765 90))
+    (property "Value" "470" (id 1) (at 173.99 26.035 90))
+    (property "Footprint" "azonenberg_pcb:EIA_0402_RES_NOSILK" (id 2) (at 173.99 27.813 90)
+      (effects (font (size 1.27 1.27)) hide)
+    )
+    (property "Datasheet" "" (id 3) (at 173.99 26.035 0)
+      (effects (font (size 1.27 1.27)) hide)
+    )
