File: oscilloscope-probing/lab/boards/prbs-generator/prbs-generator.kicad_pcb (KiCad board)
At the start: 4 copper layers, 84 parts, among them J1 BARREL_JACK, J2 HEADER_1x5, J3 32K243-40ML5, J4 32K243-40ML5, J5 HEADER_1x3, J6 HEADER_1x3, SW1 BUTTON, SW2 BUTTON, SW3 BUTTON, SW4 BUTTON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

Commit message: Continued work on PRBS board layout
Parts:
- added MH1: HOLE, azonenberg_pcb:MECHANICAL_CLEARANCEHOLE_4_40, F.Cu at (60.0, 39.8)
- added MH2: HOLE, azonenberg_pcb:MECHANICAL_CLEARANCEHOLE_4_40, F.Cu at (103.0, 118.0)
- added MH3: HOLE, azonenberg_pcb:MECHANICAL_CLEARANCEHOLE_4_40, F.Cu at (60.0, 118.0)
- added MH4: HOLE, azonenberg_pcb:MECHANICAL_CLEARANCEHOLE_4_40, F.Cu at (103.0, 39.8)
- C11, C16, C17, C7, C9, R23, R24: moved to B.Cu
- moved R4 103.5 mm to (57.8, 70.2), turned to 180 degrees
- moved R5 103.0 mm to (57.8, 72.2), turned to 180 degrees
- moved R7 102.9 mm to (57.8, 85.2), turned to 180 degrees
- moved R15 102.9 mm to (57.8, 87.2), turned to 180 degrees
- moved R18 101.5 mm to (57.8, 107.2), turned to 180 degrees
- moved R14 101.4 mm to (57.8, 83.2), turned to 180 degrees
- moved R13 100.9 mm to (57.8, 76.2), turned to 180 degrees
- moved R10 100.1 mm to (57.8, 105.2), turned to 180 degrees
- moved R12 99.0 mm to (57.8, 74.2), turned to 180 degrees
- moved D2 97.8 mm to (60.5, 72.2), turned to 180 degrees
- moved R9 97.1 mm to (57.8, 101.2), turned to 180 degrees
- moved R8 95.4 mm to (57.8, 92.2), turned to 180 degrees
- moved D8 95.0 mm to (60.5, 109.2), turned to 180 degrees
- moved R17 94.6 mm to (57.8, 103.2), turned to 180 degrees
- moved R6 94.1 mm to (57.8, 81.2), turned to 180 degrees
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- renumbered G*** to G1, G*** to G2, G*** to G3
Connections:
- U1 pad 4: (no net) -> /3V3
- U3 pad 10: Net-(D10-Pad1) -> Net-(D12-Pad1)
- U3 pad 15: Net-(D3-Pad1) -> Net-(D1-Pad1)
- U3 pad 16: Net-(D11-Pad1) -> Net-(D2-Pad1)
- U3 pad 19: Net-(D4-Pad1) -> Net-(D9-Pad1)
- U3 pad 20: Net-(D12-Pad1) -> Net-(D10-Pad1)
- U3 pad 5: Net-(D1-Pad1) -> Net-(D3-Pad1)
- U3 pad 6: Net-(D9-Pad1) -> Net-(D11-Pad1)
- U3 pad 9: Net-(D2-Pad1) -> Net-(D4-Pad1)
Routing:
- net /3V3: track 0.00 -> 290.5 mm, vias 0 -> 88
- net /GND: track 0.00 -> 228.5 mm, vias 0 -> 25
- net /I2C_SDA: track 0.00 -> 54.7 mm, vias 0 -> 3
- net /I2C_SCL: track 0.00 -> 52.5 mm, vias 0 -> 3
- net Net-(D12-Pad1): track 0.00 -> 40.0 mm
- net /NEXT_RATE: track 0.00 -> 39.0 mm, vias 0 -> 1
- net Net-(D4-Pad1): track 0.00 -> 37.0 mm
- net Net-(D11-Pad1): track 0.00 -> 32.5 mm
- net Net-(D3-Pad1): track 0.00 -> 28.8 mm
- net /NEXT_DRIVE: track 0.00 -> 28.0 mm, vias 0 -> 1
- net /PRBS Generation/OUT_AC_P: track 0.00 -> 26.1 mm
- net /PRBS Generation/OUT_AC_N: track 0.00 -> 26.1 mm
- net Net-(D1-Pad1): track 0.00 -> 25.2 mm
- net Net-(D2-Pad1): track 0.00 -> 23.5 mm
- net Net-(D9-Pad1): track 0.00 -> 23.2 mm
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- added copper zone on F.Cu, net /3V3
- added copper zone on In2.Cu, net /3V3
- added copper zone on In1.Cu, net /GND
Other:
- board outline added: 53 x 89 mm
- board text added: "+"
- board text added: "-"
- board text added: "0 dB"
- board text added: "0.9 dB"
- board text added: "1.25 Gbps"
- board text added: "10.3125 Gbps"
- board text added: "1000 mV"
- board text added: "12.0 dB"
- board text added: "1200 mV"
- board text added: "2.0 dB"
- board text added: "2.5 Gbps"
- board text added: "3.3 dB"
- board text added: "3V3"
- board text added: "5.0 Gbps"
- board text added: "5V DC"
- board text added: "6.0 dB"
- board text added: "600 mV"
- board text added: "800 mV"
- board text added: "DATA RATE"
- board text added: "DE-EMPHASIS"
- board text added: "DRIVE STRENGTH"
- board text added: "Differential"
- board text added: "GND"
- board text added: "I2C DBG"
- board text added: "PATTERN"
- board text added: "PRBS Generator v0.1 A. Zonenberg 2022-03-19"
- board text added: "PRBS31"
- board text added: "PRBS9"
- board text added: "RST#"
- board text added: "RX"
- board text added: "SCL"
- board text added: "SDA"
- board text added: "SWCLK"
- board text added: "SWD"
- board text added: "SWDIO"
- board text added: "Single ended"
- board text added: "TX"
- board text added: "UART"

Commit message: Finished initial PRBS generator
Parts:
- added C22: 4.7 uF, azonenberg_pcb:EIA_0603_CAP_NOSILK, F.Cu at (93.9, 102.6)
- added C23: 0.47 uF, azonenberg_pcb:EIA_0402_CAP_NOSILK, B.Cu at (94.2, 107.4)
- added C24: 0.47 uF, azonenberg_pcb:EIA_0402_CAP_NOSILK, B.Cu at (90.3, 107.5)
- added TP2: U.FL, azonenberg_pcb:CONN_U.FL_TE_1909763-1, F.Cu at (85.7, 70.6)
- C10, C12, C4, C8: moved to B.Cu
- moved C8 10.1 mm to (83.6, 100.8), turned to 90 degrees
- moved C12 7.54 mm to (82.4, 99.2)
- moved U2 5.84 mm to (92.2, 106.5)
- moved R2 5.82 mm to (91.8, 101.9), turned to 90 degrees
- moved R3 5.59 mm to (90.2, 102.9), turned to 90 degrees
- moved C4 5.02 mm to (88.9, 106.0), turned to 180 degrees
- moved R1 5.00 mm to (89.0, 104.5), turned to -90 degrees
- moved C10 4.10 mm to (85.1, 99.9), turned to 180 degrees
- moved C6 2.96 mm to (88.2, 98.3)
- moved U4 2.15 mm to (83.7, 99.5), turned to -90 degrees
- moved C17 0.71 mm to (81.8, 57.8)
Routing:
- net /GND: track 228.5 -> 282.2 mm, vias 25 -> 37
- net /3V3: track 290.5 -> 334.1 mm, vias 88 -> 100
- net Net-(D16-Pad1): track 0.00 -> 37.1 mm
- net Net-(D8-Pad1): track 0.00 -> 34.4 mm
- net Net-(D15-Pad1): track 0.00 -> 30.3 mm
- net Net-(D7-Pad1): track 0.00 -> 27.5 mm
- net /I2C_SCL: track 52.5 -> 79.5 mm, vias 3 -> 5
- net Net-(D5-Pad1): track 0.00 -> 24.5 mm
- net Net-(D13-Pad1): track 0.00 -> 22.7 mm
- net /UART_TX: track 0.00 -> 22.4 mm, vias 0 -> 1
- net /I2C_SDA: track 54.7 -> 77.0 mm, vias 3 -> 5
- net Net-(D14-Pad1): track 0.00 -> 22.1 mm
- net /NEXT_EMPH: track 8.07 -> 30.1 mm, vias 1 -> 2
- net Net-(D6-Pad1): track 0.00 -> 21.4 mm
- net /UART_RX: track 0.00 -> 19.5 mm, vias 0 -> 1
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Other:
- board text added: "PRBS Generator v0.1 A. Zonenberg 2022-03-20"
- board text removed: "PRBS Generator v0.1 A. Zonenberg 2022-03-19"
