File: oscilloscope-probing/lab/boards/prbs-generator/prbs-generator.kicad_sch (KiCad schematic)
At the start: 20 parts, among them J1 BARREL_JACK, J2 HEADER_1x5, J5 HEADER_1x3, J6 HEADER_1x3, SW1 BUTTON, SW2 BUTTON, SW3 BUTTON, SW4 BUTTON, U1 ZLDO1117-33, U2 STM32F031-QFN28

Commit message: Continued work on PRBS board layout
Parts:
- added MH1, MH2, MH3, MH4: HOLE, azonenberg_pcb:MECHANICAL_CLEARANCEHOLE_4_40, symbol conn:CONN_01X01
- U1: symbol power-azonenberg:LDO1117-XX -> power-azonenberg:LDO1117-XX_SOT223
Connections:
- net 3V3: now also U1.4 (Vout)
- no-connect marks 14 -> 18
Other:
- moved on the sheet: C3
Changed lines of the file:
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@@
   (title_block
     (title "PRBS Generator")
-    (date "2022-03-18")
+    (date "2022-03-19")
     (rev "0.1")
     (company "Antikernel Labs")
@@
   (junction (at 77.47 20.955) (diameter 0) (color 0 0 0 0)
   )
-  (junction (at 125.73 20.955) (diameter 0) (color 0 0 0 0)
+  (junction (at 113.03 20.955) (diameter 0) (color 0 0 0 0)
+  )
+  (junction (at 106.68 20.955) (diameter 0) (color 0 0 0 0)
   )
   (junction (at 67.945 20.955) (diameter 0) (color 0 0 0 0)
   )
+  (no_connect (at 22.86 77.47))
   (no_connect (at 234.95 146.685))
   (no_connect (at 234.95 144.145))
@@
   (no_connect (at 234.95 66.04))
   (no_connect (at 234.95 114.3))
+  (no_connect (at 234.95 96.52))
   (no_connect (at 234.95 99.06))
   (no_connect (at 234.95 101.6))
-  (no_connect (at 234.95 96.52))
+  (no_connect (at 22.86 69.215))
+  (no_connect (at 22.86 52.705))
   (no_connect (at 29.21 26.035))
+  (no_connect (at 22.86 60.96))
   (wire (pts (xy 29.21 20.955) (xy 34.925 20.955))
     (stroke (width 0) (type default) (color 0 0 0 0))
   )
-  (wire (pts (xy 125.73 20.955) (xy 134.62 20.955))
+  (wire (pts (xy 113.03 20.955) (xy 121.92 20.955))
     (stroke (width 0) (type default) (color 0 0 0 0))
   )
@@
     (stroke (width 0) (type default) (color 0 0 0 0))
   )
-  (wire (pts (xy 125.73 28.575) (xy 134.62 28.575))
+  (wire (pts (xy 113.03 28.575) (xy 121.92 28.575))
     (stroke (width 0) (type default) (color 0 0 0 0))
   )
@@
     (stroke (width 0) (type default) (color 0 0 0 0))
   )
+  (wire (pts (xy 106.68 20.955) (xy 106.68 23.495))
+    (stroke (width 0) (type default) (color 0 0 0 0))
+  )
+  (wire (pts (xy 113.03 20.955) (xy 106.68 20.955))
+    (stroke (width 0) (type default) (color 0 0 0 0))
+  )
   (wire (pts (xy 57.15 20.955) (xy 67.945 20.955))
     (stroke (width 0) (type default) (color 0 0 0 0))
@@
     (stroke (width 0) (type default) (color 0 0 0 0))
   )
+  (wire (pts (xy 91.44 28.575) (xy 93.98 28.575))
+    (stroke (width 0) (type default) (color 0 0 0 0))
+  )
   (label "NEXT_PAT" (at 267.97 140.97 0)
     (effects (font (size 1.27 1.27)) (justify left bottom))
@@
     (effects (font (size 1.27 1.27)) (justify left bottom))
   )
-  (label "GND" (at 134.62 28.575 0)
+  (label "GND" (at 121.92 28.575 0)
     (effects (font (size 1.27 1.27)) (justify left bottom))
   )
@@
     (effects (font (size 1.27 1.27)) (justify right bottom))
   )
-  (label "3V3" (at 134.62 20.955 0)
+  (label "3V3" (at 121.92 20.955 0)
     (effects (font (size 1.27 1.27)) (justify left bottom))
   )
@@
     (effects (font (size 1.27 1.27)) (justify right bottom))
   )
-  (label "GND" (at 104.14 34.925 180)
+  (label "GND" (at 91.44 28.575 180)
     (effects (font (size 1.27 1.27)) (justify right bottom))
   )
@@
     (pin "1")
     (pin "2")
+  )
+  (symbol (lib_id "conn:CONN_01X01") (at 27.94 69.215 0) (unit 1)
+    (in_bom yes) (on_board yes)
+    (property "Reference" "MH3" (id 0) (at 27.94 66.675 0))
+    (property "Value" "HOLE" (id 1) (at 27.94 72.39 0))
+    (property "Footprint" "azonenberg_pcb:MECHANICAL_CLEARANCEHOLE_4_40" (id 2) (at 27.94 69.215 0)
+      (effects (font (size 1.27 1.27)) hide)
+    )
+    (property "Datasheet" "" (id 3) (at 27.94 69.215 0)
+      (effects (font (size 1.27 1.27)) hide)
+    )
+    (pin "1")
+  )
+  (symbol (lib_id "conn:CONN_01X01") (at 27.94 60.96 0) (unit 1)
+    (in_bom yes) (on_board yes)
+    (property "Reference" "MH2" (id 0) (at 27.94 58.42 0))
+    (property "Value" "HOLE" (id 1) (at 27.94 64.135 0))
+    (property "Footprint" "azonenberg_pcb:MECHANICAL_CLEARANCEHOLE_4_40" (id 2) (at 27.94 60.96 0)
+      (effects (font (size 1.27 1.27)) hide)
+    )
+    (property "Datasheet" "" (id 3) (at 27.94 60.96 0)
+      (effects (font (size 1.27 1.27)) hide)
+    )
+    (pin "1")
   )
   (symbol (lib_id "st-azonenberg:STM32F031-QFN28") (at 237.49 115.57 0) (unit 2)
@@
     (pin "3")
   )
-  (symbol (lib_id "power-azonenberg:LDO1117-XX") (at 102.87 18.415 0) (unit 1)
-    (in_bom yes) (on_board yes)
-    (property "Reference" "U1" (id 0) (at 104.14 18.415 0)
+  (symbol (lib_id "power-azonenberg:LDO1117-XX_SOT223") (at 93.98 18.415 0) (unit 1)
+    (in_bom yes) (on_board yes)
+    (property "Reference" "U1" (id 0) (at 106.045 17.78 0)
       (effects (font (size 1.524 1.524)))
     )
-    (property "Value" "ZLDO1117-33" (id 1) (at 113.03 29.21 0)
+    (property "Value" "ZLDO1117-33" (id 1) (at 94.615 17.145 0)
       (effects (font (size 1.524 1.524)))
     )
-    (property "Footprint" "azonenberg_pcb:SOT223-4" (id 2) (at 102.87 18.415 0)
+    (property "Footprint" "azonenberg_pcb:SOT223-4" (id 2) (at 93.98 15.875 0)
       (effects (font (size 1.524 1.524)) hide)
     )
-    (property "Datasheet" "" (id 3) (at 102.87 18.415 0)
+    (property "Datasheet" "" (id 3) (at 93.98 18.415 0)
       (effects (font (size 1.524 1.524)))
     )
@@
     (pin "2")
     (pin "3")
+    (pin "4")
   )
   (symbol (lib_id "device:R") (at 261.62 55.88 90) (unit 1)
@@
     (pin "2")
   )
-  (symbol (lib_id "device:C") (at 125.73 24.765 0) (unit 1)
-    (in_bom yes) (on_board yes)
-    (property "Reference" "C3" (id 0) (at 126.365 22.225 0)
-      (effects (font (size 1.27 1.27)) (justify left))
-    )
-    (property "Value" "4.7 uF" (id 1) (at 126.365 27.305 0)
-      (effects (font (size 1.27 1.27)) (justify left))
-    )
-    (property "Footprint" "azonenberg_pcb:EIA_0603_CAP_NOSILK" (id 2) (at 126.6952 28.575 0)
-      (effects (font (size 1.27 1.27)) hide)
-    )
-    (property "Datasheet" "" (id 3) (at 125.73 24.765 0)
+  (symbol (lib_id "device:C") (at 113.03 24.765 0) (unit 1)
+    (in_bom yes) (on_board yes)
+    (property "Reference" "C3" (id 0) (at 113.665 22.225 0)
+      (effects (font (size 1.27 1.27)) (justify left))
+    )
+    (property "Value" "4.7 uF" (id 1) (at 113.665 27.305 0)
+      (effects (font (size 1.27 1.27)) (justify left))
+    )
+    (property "Footprint" "azonenberg_pcb:EIA_0603_CAP_NOSILK" (id 2) (at 113.9952 28.575 0)
+      (effects (font (size 1.27 1.27)) hide)
+    )
+    (property "Datasheet" "" (id 3) (at 113.03 24.765 0)
       (effects (font (size 1.27 1.27)) hide)
     )
@@
     (pin "4")
     (pin "5")
+  )
+  (symbol (lib_id "conn:CONN_01X01") (at 27.94 52.705 0) (unit 1)
+    (in_bom yes) (on_board yes)
+    (property "Reference" "MH1" (id 0) (at 27.94 50.165 0))
+    (property "Value" "HOLE" (id 1) (at 27.94 55.88 0))
+    (property "Footprint" "azonenberg_pcb:MECHANICAL_CLEARANCEHOLE_4_40" (id 2) (at 27.94 52.705 0)
+      (effects (font (size 1.27 1.27)) hide)
+    )
+    (property "Datasheet" "" (id 3) (at 27.94 52.705 0)
+      (effects (font (size 1.27 1.27)) hide)
+    )
+    (pin "1")
+  )
+  (symbol (lib_id "conn:CONN_01X01") (at 27.94 77.47 0) (unit 1)
+    (in_bom yes) (on_board yes)
+    (property "Reference" "MH4" (id 0) (at 27.94 74.93 0))
+    (property "Value" "HOLE" (id 1) (at 27.94 80.645 0))
+    (property "Footprint" "azonenberg_pcb:MECHANICAL_CLEARANCEHOLE_4_40" (id 2) (at 27.94 77.47 0)
+      (effects (font (size 1.27 1.27)) hide)
+    )
+    (property "Datasheet" "" (id 3) (at 27.94 77.47 0)
+      (effects (font (size 1.27 1.27)) hide)
+    )
+    (pin "1")
   )
   (symbol (lib_id "conn:CONN_01X03") (at 269.24 111.76 0) (unit 1)
@@
       (reference "J6") (unit 1) (value "HEADER_1x3") (footprint "azonenberg_pcb:CONN_HEADER_2.54MM_1x3")
     )
+    (path "/f15cbf5d-7b4a-4057-9b8c-17709b18a88a"
+      (reference "MH1") (unit 1) (value "HOLE") (footprint "azonenberg_pcb:MECHANICAL_CLEARANCEHOLE_4_40")
+    )
+    (path "/76b83de5-f75d-4b59-a5dc-d8d5fa98775a"
+      (reference "MH2") (unit 1) (value "HOLE") (footprint "azonenberg_pcb:MECHANICAL_CLEARANCEHOLE_4_40")
+    )
+    (path "/6ae37ca5-3566-47a5-9ac3-c09c03381faa"
+      (reference "MH3") (unit 1) (value "HOLE") (footprint "azonenberg_pcb:MECHANICAL_CLEARANCEHOLE_4_40")
+    )
+    (path "/f8fc8929-4928-4cc0-9b0b-2ccef4d059b1"
+      (reference "MH4") (unit 1) (value "HOLE") (footprint "azonenberg_pcb:MECHANICAL_CLEARANCEHOLE_4_40")
+    )
     (path "/d7a5d784-52e3-4d8d-a227-33afec8ed180"

Commit message: Finished initial PRBS generator
Parts:
- added C22: 4.7 uF, azonenberg_pcb:EIA_0603_CAP_NOSILK, symbol device:C
- added C23, C24: 0.47 uF, azonenberg_pcb:EIA_0402_CAP_NOSILK, symbol device:C
- added TP2: U.FL, azonenberg_pcb:CONN_U.FL_TE_1909763-1, symbol conn:CONN_COAXIAL
Connections:
- net 3V3: now also C22.1, C23.1, C24.1, TP2.1 (In)
- net GND: now also C22.2, C23.2, C24.2, TP2.2 (Ext)
Changed lines of the file:
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@@
   (title_block
     (title "PRBS Generator")
-    (date "2022-03-19")
+    (date "2022-03-20")
     (rev "0.1")
     (company "Antikernel Labs")
@@
   (junction (at 77.47 20.955) (diameter 0) (color 0 0 0 0)
   )
+  (junction (at 199.39 126.365) (diameter 0) (color 0 0 0 0)
+  )
   (junction (at 113.03 20.955) (diameter 0) (color 0 0 0 0)
   )
+  (junction (at 186.055 133.985) (diameter 0) (color 0 0 0 0)
+  )
   (junction (at 106.68 20.955) (diameter 0) (color 0 0 0 0)
+  )
+  (junction (at 186.055 126.365) (diameter 0) (color 0 0 0 0)
   )
   (junction (at 67.945 20.955) (diameter 0) (color 0 0 0 0)
@@
     (stroke (width 0) (type default) (color 0 0 0 0))
   )
-  (wire (pts (xy 231.14 126.365) (xy 234.95 126.365))
+  (wire (pts (xy 199.39 126.365) (xy 234.95 126.365))
+    (stroke (width 0) (type default) (color 0 0 0 0))
+  )
+  (wire (pts (xy 175.26 126.365) (xy 186.055 126.365))
+    (stroke (width 0) (type default) (color 0 0 0 0))
+  )
+  (wire (pts (xy 186.055 126.365) (xy 199.39 126.365))
+    (stroke (width 0) (type default) (color 0 0 0 0))
+  )
+  (wire (pts (xy 186.055 133.985) (xy 199.39 133.985))
     (stroke (width 0) (type default) (color 0 0 0 0))
   )
@@
   )
   (wire (pts (xy 57.15 20.955) (xy 67.945 20.955))
+    (stroke (width 0) (type default) (color 0 0 0 0))
+  )
+  (wire (pts (xy 175.26 133.985) (xy 186.055 133.985))
     (stroke (width 0) (type default) (color 0 0 0 0))
   )
@@
     (effects (font (size 1.27 1.27)) (justify right bottom))
   )
+  (label "GND" (at 83.82 48.26 0)
+    (effects (font (size 1.27 1.27)) (justify left bottom))
+  )
+  (label "3V3" (at 80.01 43.18 180)
+    (effects (font (size 1.27 1.27)) (justify right bottom))
+  )
   (label "I2C_SCL" (at 234.95 68.58 180)
     (effects (font (size 1.27 1.27)) (justify right bottom))
@@
     (effects (font (size 1.27 1.27)) (justify right bottom))
   )
+  (label "GND" (at 175.26 133.985 180)
+    (effects (font (size 1.27 1.27)) (justify right bottom))
+  )
   (label "UART_RX" (at 234.95 106.68 180)
     (effects (font (size 1.27 1.27)) (justify right bottom))
@@
     (effects (font (size 1.27 1.27)) (justify right bottom))
   )
-  (label "3V3" (at 231.14 126.365 180)
+  (label "3V3" (at 175.26 126.365 180)
     (effects (font (size 1.27 1.27)) (justify right bottom))
   )
@@
     )
     (property "Datasheet" "" (id 3) (at 67.945 24.765 0)
+      (effects (font (size 1.27 1.27)) hide)
+    )
+    (pin "1")
+    (pin "2")
+  )
+  (symbol (lib_id "device:C") (at 186.055 130.175 0) (unit 1)
+    (in_bom yes) (on_board yes) (fields_autoplaced)
+    (property "Reference" "C23" (id 0) (at 188.976 129.2665 0)
+      (effects (font (size 1.27 1.27)) (justify left))
+    )
+    (property "Value" "0.47 uF" (id 1) (at 188.976 132.0416 0)
+      (effects (font (size 1.27 1.27)) (justify left))
+    )
+    (property "Footprint" "azonenberg_pcb:EIA_0402_CAP_NOSILK" (id 2) (at 187.0202 133.985 0)
+      (effects (font (size 1.27 1.27)) hide)
+    )
+    (property "Datasheet" "" (id 3) (at 186.055 130.175 0)
       (effects (font (size 1.27 1.27)) hide)
     )
@@
     )
     (pin "1")
+  )
+  (symbol (lib_id "device:C") (at 199.39 130.175 0) (unit 1)
+    (in_bom yes) (on_board yes) (fields_autoplaced)
+    (property "Reference" "C24" (id 0) (at 202.311 129.2665 0)
+      (effects (font (size 1.27 1.27)) (justify left))
+    )
+    (property "Value" "0.47 uF" (id 1) (at 202.311 132.0416 0)
+      (effects (font (size 1.27 1.27)) (justify left))
+    )
+    (property "Footprint" "azonenberg_pcb:EIA_0402_CAP_NOSILK" (id 2) (at 200.3552 133.985 0)
+      (effects (font (size 1.27 1.27)) hide)
+    )
+    (property "Datasheet" "" (id 3) (at 199.39 130.175 0)
+      (effects (font (size 1.27 1.27)) hide)
+    )
+    (pin "1")
+    (pin "2")
   )
   (symbol (lib_id "st-azonenberg:STM32F031-QFN28") (at 237.49 115.57 0) (unit 2)
@@
     (pin "3")
   )
+  (symbol (lib_id "conn:CONN_COAXIAL") (at 83.82 43.18 0) (unit 1)
+    (in_bom yes) (on_board yes)
+    (property "Reference" "TP2" (id 0) (at 84.074 40.132 0))
+    (property "Value" "U.FL" (id 1) (at 86.741 43.18 90))
+    (property "Footprint" "azonenberg_pcb:CONN_U.FL_TE_1909763-1" (id 2) (at 83.82 43.18 0)
+      (effects (font (size 1.27 1.27)) hide)
+    )
+    (property "Datasheet" "" (id 3) (at 83.82 43.18 0)
+      (effects (font (size 1.27 1.27)) hide)
+    )
+    (pin "1")
+    (pin "2")
+  )
+  (symbol (lib_id "device:C") (at 175.26 130.175 0) (unit 1)
+    (in_bom yes) (on_board yes)
+    (property "Reference" "C22" (id 0) (at 175.895 127.635 0)
+      (effects (font (size 1.27 1.27)) (justify left))
+    )
+    (property "Value" "4.7 uF" (id 1) (at 175.895 132.715 0)
+      (effects (font (size 1.27 1.27)) (justify left))
+    )
+    (property "Footprint" "azonenberg_pcb:EIA_0603_CAP_NOSILK" (id 2) (at 176.2252 133.985 0)
+      (effects (font (size 1.27 1.27)) hide)
+    )
+    (property "Datasheet" "" (id 3) (at 175.26 130.175 0)
+      (effects (font (size 1.27 1.27)) hide)
+    )
+    (pin "1")
+    (pin "2")
+  )
   (symbol (lib_id "power-azonenberg:LDO1117-XX_SOT223") (at 93.98 18.415 0) (unit 1)
     (in_bom yes) (on_board yes)
@@
       (reference "C21") (unit 1) (value "0.1 uF") (footprint "azonenberg_pcb:EIA_0402_CAP_NOSILK")
     )
+    (path "/b505bb24-da6f-4fad-a897-730f4a13caa4"
+      (reference "C22") (unit 1) (value "4.7 uF") (footprint "azonenberg_pcb:EIA_0603_CAP_NOSILK")
+    )
+    (path "/23fde716-4b8d-44ac-b4f3-8a9a4d52d3f9"
+      (reference "C23") (unit 1) (value "0.47 uF") (footprint "azonenberg_pcb:EIA_0402_CAP_NOSILK")
+    )
+    (path "/7acbcf15-5a60-4e68-97b1-5dd77eabd674"
+      (reference "C24") (unit 1) (value "0.47 uF") (footprint "azonenberg_pcb:EIA_0402_CAP_NOSILK")
+    )
     (path "/1914c7dd-0b8e-4406-b7dd-046aeb1e19a9/88b62a79-7e7f-4309-b8f3-68ce12a1f2c5"
       (reference "D1") (unit 1) (value "GREEN") (footprint "azonenberg_pcb:EIA_0805_LED")
@@
       (reference "TP1") (unit 1) (value "GNDCLIP") (footprint "azonenberg_pcb:TESTPOINT_SMT_KEYSTONE_5016")
     )
+    (path "/b2f6eda0-0062-4f47-8a2c-4b6f75b63178"
+      (reference "TP2") (unit 1) (value "U.FL") (footprint "azonenberg_pcb:CONN_U.FL_TE_1909763-1")
+    )
     (path "/ba649285-d524-479d-829f-70d8e8510aca"
