File: oscilloscope-probing/lab/boards/prbs-generator/prbs.kicad_sch (KiCad schematic)
At the start: 19 parts, among them J3 32K243-40ML5, J4 32K243-40ML5, U5 50-ECS2016MVQ-250-CN-TR, U6 DS125DF111

Commit message: Continued work on PRBS board layout
Other:
- company: (none) -> Antikernel Labs
- title: (none) -> PRBS Generator
Changed lines of the file:
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@@
 (kicad_sch (version 20211123) (generator eeschema)
   (paper "A4")
+  (title_block
+    (title "PRBS Generator")
+    (date "2022-03-19")
+    (rev "0.1")
+    (company "Antikernel Labs")
+    (comment 1 "Andrew D. Zonenberg")
+  )
   (junction (at 76.2 105.41) (diameter 0) (color 0 0 0 0)
   )
