File: oscilloscope-probing/lab/boards/demo-board/demo-board.kicad_pcb (KiCad board)
At the start: 8 copper layers, 126 x 117 mm, 304 parts, among them J1 CONN_01X03, J10 SMA-J-P-H-ST-EM1, J11 TESTCLIP, J12 TESTCLIP, J13 TESTCLIP, J14 USB_C_Receptacle_USB2.0, J15 TESTCLIP, J16 SMA-J-P-H-ST-EM1, J17 SMA-J-P-H-ST-EM1, J18 SMA-J-P-H-ST-EM1, J19 SMA-J-P-H-ST-EM1, J2 CORTEX_DEBUG_ETM, J20 SMA-J-P-H-ST-EM1, J21 SMA-J-P-H-ST-EM1, J22 SMA-J-P-H-ST-EM1, J23 SMA-J-P-H-ST-EM1, J24 PMOD_HOST, J25 PMOD_HOST, J3 XILINX_JTAG, J4 CORTEX_DEBUG_ETM, J5 DISPLAY, J6 CONN_01X06, J7 SMA-J-P-H-ST-EM1, J8 SMA-J-P-H-ST-EM1, J9 SMA-J-P-H-ST-EM1, M1 LOGO, M2 LOGO, M3 LOGO, M4 LOGO, Q1 SSM6N58NU, SW1 SWITCH, SW2 SWITCH, SW3 SWITCH, SW4 SWITCH, SW5 SWITCH, SW6 SWITCH, SW7 SWITCH, U1 FT234XD, U10 19-C47/RSGHBHC-5V01/2T, U11 19-C47/RSGHBHC-5V01/2T, U12 19-C47/RSGHBHC-5V01/2T, U13 19-C47/RSGHBHC-5V01/2T, U2 STM32L431-QFN48, U26 74LVC1T45, U3 LTC3374A, U39 NCP45525IMNTWG-H, U4 XC7A35T-2FGG484I, U5 STM32H750XBH6, U6 ECS-1612MV-250-CN, U7 ECS-1612MV-250-CN, U8 S25FL064LABMFI013, U9 SIT9121AI-2BF-XXS156.250000G

Commit message: Continued layout
Parts:
- C25, C32, C33, C40, C41: moved to B.Cu
- moved TP4 123.0 mm to (45.2, 81.5), turned to 90 degrees
- moved C25 110.3 mm to (53.5, 63.0), turned to 180 degrees
- moved C40 108.9 mm to (54.5, 76.0), turned to 180 degrees
- moved C32 107.1 mm to (56.5, 67.0)
- moved C41 106.5 mm to (58.5, 73.0)
- moved C33 103.3 mm to (59.5, 76.0)
- moved TP17 98.0 mm to (101.0, 32.2)
- moved R54 97.6 mm to (49.0, 69.0)
- moved R57 96.9 mm to (49.0, 72.0), turned to 0 degrees
- moved R55 95.7 mm to (49.0, 70.0)
- moved R56 95.2 mm to (49.0, 71.0), turned to 0 degrees
- moved TP16 83.1 mm to (117.0, 32.2)
- moved TP5 50.9 mm to (117.8, 78.2), turned to 90 degrees
- moved TP15 1.25 mm to (99.0, 39.2)
Connections:
- R54 pad 2: Net-(U4G-IO_L1P_T0_34) -> Net-(U4G-IO_L3N_T0_DQS_34)
- R55 pad 2: Net-(U4G-IO_L1N_T0_34) -> Net-(U4G-IO_L1P_T0_34)
- R56 pad 2: Net-(U4G-IO_L2P_T0_34) -> Net-(U4G-IO_L1N_T0_34)
- U4 pad B21: unconnected-(U4F-IO_L21P_T3_DQS_16-PadB21) -> /Test signals/LED_CTRL
- U4 pad F21: /Test signals/LED_CTRL -> unconnected-(U4F-IO_25_16-PadF21)
- U4 pad R2: unconnected-(U4G-IO_L3N_T0_DQS_34-PadR2) -> Net-(U4G-IO_L3N_T0_DQS_34)
- U4 pad U2: Net-(U4G-IO_L2P_T0_34) -> unconnected-(U4G-IO_L2P_T0_34-PadU2)
- U5 pad C1: /MCU/MCU_TRIG -> unconnected-(U5C-PC15-PadC1)
- U5 pad D6: unconnected-(U5G-PG15-PadD6) -> /MCU/MCU_TRIG
- U5 pad E2: unconnected-(U5I-PI9-PadE2) -> /MCU/MCU_PMOD_DQ2
- U5 pad E3: unconnected-(U5C-PC13-PadE3) -> /MCU/MCU_PMOD_DQ3
- U5 pad F3: unconnected-(U5I-PI10-PadF3) -> /MCU/MCU_PMOD_DQ6
- U5 pad G1: unconnected-(U5F-PF2-PadG1) -> /MCU/MCU_PMOD_DQ5
- U5 pad G3: unconnected-(U5F-PF1-PadG3) -> /MCU/MCU_PMOD_DQ1
- U5 pad H1: unconnected-(U5I-PI12-PadH1) -> /MCU/MCU_PMOD_DQ4
- U5 pad H2: unconnected-(U5I-PI13-PadH2) -> /MCU/MCU_PMOD_DQ0
- U5 pad H3: unconnected-(U5I-PI14-PadH3) -> /MCU/MCU_PMOD_DQ7
- U5 pad N2: /MCU/MCU_PMOD_DQ5 -> unconnected-(U5H-PH2-PadN2)
- U5 pad P2: /MCU/MCU_PMOD_DQ6 -> unconnected-(U5H-PH3-PadP2)
- U5 pad P3: /MCU/MCU_PMOD_DQ7 -> unconnected-(U5H-PH4-PadP3)
- U5 pad R3: /MCU/MCU_PMOD_DQ4 -> unconnected-(U5A-PA6-PadR3)
- U5 pad T4: /MCU/MCU_PMOD_DQ3 -> unconnected-(U5C-PC4-PadT4)
- U5 pad T5: /MCU/MCU_PMOD_DQ1 -> unconnected-(U5B-PB1-PadT5)
- U5 pad U2: /MCU/MCU_PMOD_DQ2 -> unconnected-(U5A-PA3-PadU2)
- U5 pad U4: /MCU/MCU_PMOD_DQ0 -> unconnected-(U5C-PC5-PadU4)
Routing:
- net /Test signals/COAX_1: track 0.00 -> 135.3 mm, vias 0 -> 2
- net /Test signals/COAX_2: track 0.00 -> 119.7 mm, vias 0 -> 2
- net /Test signals/COAX_4: track 0.00 -> 116.6 mm, vias 0 -> 2
- net /Test signals/COAX_3: track 0.00 -> 105.0 mm, vias 0 -> 2
- net /MCU/MCU_PMOD_DQ7: track 0.00 -> 63.5 mm, vias 0 -> 1
- net /MCU/MCU_PMOD_DQ6: track 0.00 -> 58.6 mm
- net /MCU/MCU_PMOD_DQ5: track 0.00 -> 56.7 mm
- net /MCU/MCU_PMOD_DQ4: track 0.00 -> 56.1 mm
- net /MCU/MCU_PMOD_DQ3: track 5.30 -> 59.3 mm, vias 0 -> 1
- net /Test signals/GTP_TX1_P: track 0.00 -> 54.0 mm, vias 1 -> 0
- net /Test signals/GTP_TX1_N: track 0.00 -> 53.7 mm, vias 1 -> 0
- net /Test signals/GTP_TX0_N: track 0.00 -> 53.7 mm, vias 1 -> 0
- net /Test signals/2XTHRU: track 0.00 -> 53.7 mm
- net /Test signals/GTP_TX0_P: track 0.00 -> 53.6 mm, vias 1 -> 0
- net /MCU/MCU_PMOD_DQ2: track 2.97 -> 54.8 mm
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Other:
- board text added: "1V8"
- board text added: "DAC1"
- board text added: "DAC2"
- board text added: "GTP0_N"
- board text added: "GTP0_P"
- board text added: "GTP1_N"
- board text added: "GTP1_P"
- board text removed: "1V0"
