File: oscilloscope-probing/lab/boards/demo-board/demo-board.kicad_sch (KiCad schematic)
At the start: 4 parts

Commit message: Finished initial demo board schematic
Parts:
- added MH1, MH2, MH3, MH4: 4-40, symbol special-azonenberg:MECHANICAL
Other:
- sheet MCU ports: added DAC1_OUT1, DAC1_OUT2; removed none
- sheet Test signals ports: added 3V3, DAC1_OUT1, DAC1_OUT2, GND, GTP_VTT, VBUS; removed none

Commit message: Continued initial schematic, assigned footprints
Parts:
- MH1, MH2, MH3, MH4: footprint (none) -> azonenberg_pcb:MECHANICAL_CLEARANCEHOLE_4_40
- R22, R23, R24, R25: footprint (none) -> azonenberg_pcb:EIA_0402_RES_NOSILK
Changed lines of the file:
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@@
 			)
 		)
-		(property "Footprint" ""
+		(property "Footprint" "azonenberg_pcb:EIA_0402_RES_NOSILK"
 			(at 39.37 69.088 90)
 			(effects
@@
 			)
 		)
-		(property "Footprint" ""
+		(property "Footprint" "azonenberg_pcb:MECHANICAL_CLEARANCEHOLE_4_40"
 			(at 16.51 91.44 0)
 			(effects
@@
 			)
 		)
-		(property "Footprint" ""
+		(property "Footprint" "azonenberg_pcb:MECHANICAL_CLEARANCEHOLE_4_40"
 			(at 16.51 97.79 0)
 			(effects
@@
 			)
 		)
-		(property "Footprint" ""
+		(property "Footprint" "azonenberg_pcb:EIA_0402_RES_NOSILK"
 			(at 39.37 74.168 90)
 			(effects
@@
 			)
 		)
-		(property "Footprint" ""
+		(property "Footprint" "azonenberg_pcb:EIA_0402_RES_NOSILK"
 			(at 39.37 71.628 90)
 			(effects
@@
 			)
 		)
-		(property "Footprint" ""
+		(property "Footprint" "azonenberg_pcb:MECHANICAL_CLEARANCEHOLE_4_40"
 			(at 16.51 104.14 0)
 			(effects
@@
 			)
 		)
-		(property "Footprint" ""
+		(property "Footprint" "azonenberg_pcb:MECHANICAL_CLEARANCEHOLE_4_40"
 			(at 16.51 85.09 0)
 			(effects
@@
 			)
 		)
-		(property "Footprint" ""
+		(property "Footprint" "azonenberg_pcb:EIA_0402_RES_NOSILK"
 			(at 39.37 76.708 90)
 			(effects

Commit message: Continued demo board layout
Parts:
- added FID1, FID2, FID3, FID4, FID5, FID6: FIDUCIAL, azonenberg_pcb:FIDUCIAL_1MM, symbol special-azonenberg:MECHANICAL
- added M1: LOGO, azonenberg_pcb:LONGTHING-1200DPI, symbol special-azonenberg:MECHANICAL
- added M2: LOGO, w_logo:Logo_silk_ROHS_5x2.8mm, symbol special-azonenberg:MECHANICAL
- added M3: LOGO, w_logo:Logo_silk_WEEE_3.4x5mm, symbol special-azonenberg:MECHANICAL
- added M4: LOGO, w_logo:Logo_silk_OSHW_6x6mm, symbol special-azonenberg:MECHANICAL

Commit message: Continued demo board layout
Other:
- company: (none) -> Antikernel Labs
- title: (none) -> Oscilloscope Demo Board
Changed lines of the file:
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@@
 	(generator_version "9.0")
 	(paper "A3")
+	(title_block
+		(title "Oscilloscope Demo Board")
+		(date "2026-08-08")
+		(rev "0.1")
+		(company "Antikernel Labs")
+		(comment 1 "Andrew D. Zonenberg")
+	)
 	(wire
 		(pts
