File: oscilloscope-probing/lab/boards/demo-board/display.kicad_sch (KiCad schematic)
At the start: 19 parts, among them J5 DISPLAY, Q1 SSM6N58NU

Commit message: Continued demo board layout
Connections:
- net DPY_BS: now also TP14.7 (P7); no longer TP14.5 (P5)
- net DPY_BUSY_N: now also TP14.6 (P6); no longer TP14.7 (P7)
- net DPY_DC: now also TP14.4 (P4); no longer TP14.1 (P1)
- net DPY_RST_N: now also TP14.5 (P5); no longer TP14.4 (P4)
- net DPY_SPI_CS_N: now also TP14.3 (P3); no longer TP14.6 (P6)
- net DPY_SPI_DATA: now also TP14.1 (P1); no longer TP14.3 (P3)
Changed lines of the file:
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@@
 	)
 	(label "DPY_BUSY_N"
-		(at 41.91 40.64 180)
+		(at 41.91 38.1 180)
 		(effects
 			(font
@@
 	)
 	(label "DPY_SPI_CS_N"
-		(at 41.91 38.1 180)
+		(at 41.91 30.48 180)
 		(effects
 			(font
@@
 	)
 	(label "DPY_RST_N"
-		(at 41.91 33.02 180)
+		(at 41.91 35.56 180)
 		(effects
 			(font
@@
 	)
 	(label "DPY_DC"
-		(at 41.91 25.4 180)
+		(at 41.91 33.02 180)
 		(effects
 			(font
@@
 	)
 	(label "DPY_SPI_DATA"
-		(at 41.91 30.48 180)
+		(at 41.91 25.4 180)
 		(effects
 			(font
@@
 	)
 	(label "DPY_BS"
-		(at 41.91 35.56 180)
+		(at 41.91 40.64 180)
 		(effects
 			(font

Commit message: Continued demo board layout
Other:
- company: (none) -> Antikernel Labs
- title: (none) -> Oscilloscope Demo Board
Changed lines of the file:
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@@
 	(generator_version "9.0")
 	(paper "A3")
+	(title_block
+		(title "Oscilloscope Demo Board")
+		(date "2026-08-08")
+		(rev "0.1")
+		(company "Antikernel Labs")
+		(comment 1 "Andrew D. Zonenberg")
+	)
 	(junction
 		(at 105.41 147.32)
