File: oscilloscope-probing/lab/boards/demo-board/psu.kicad_sch (KiCad schematic)
At the start: 65 parts, among them J1 CONN_01X03, J2 CORTEX_DEBUG_ETM, SW1 SWITCH, SW2 SWITCH, U2 STM32L431-QFN48, U3 LTC3374A

Commit message: Finished initial routing of demo board but might still add more features
Connections:
- net 3V3_SW: now reaches L4.2, U3.28 (SW7), U3.29 (SW8)
Changed lines of the file:
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@@
 	(title_block
 		(title "Oscilloscope Demo Board")
-		(date "2026-08-12")
+		(date "2026-08-13")
 		(rev "0.1")
 		(company "Antikernel Labs")
@@
 		(effects
 			(font
+				(size 1.27 1.27)
+			)
+			(justify left bottom)
+		)
+	)
+	(label "3V3_SW"
+		(at 66.04 123.19 0)
+		(effects
+			(font
