File: oscilloscope-probing/lab/boards/demo-board/testsignals.kicad_sch (KiCad schematic)
At the start: 53 parts, among them J10 SMA-J-P-H-ST-EM1, J11 TESTCLIP, J12 TESTCLIP, J13 TESTCLIP, J15 TESTCLIP, J16 SMA-J-P-H-ST-EM1, J17 SMA-J-P-H-ST-EM1, J18 SMA-J-P-H-ST-EM1, J19 SMA-J-P-H-ST-EM1, J20 SMA-J-P-H-ST-EM1, J21 SMA-J-P-H-ST-EM1, J22 SMA-J-P-H-ST-EM1, J23 SMA-J-P-H-ST-EM1, J6 CONN_01X06, J7 SMA-J-P-H-ST-EM1, J8 SMA-J-P-H-ST-EM1, J9 SMA-J-P-H-ST-EM1, U10 19-C47/RSGHBHC-5V01/2T, U11 19-C47/RSGHBHC-5V01/2T, U12 19-C47/RSGHBHC-5V01/2T, U13 19-C47/RSGHBHC-5V01/2T, U26 74LVC1T45, U4 XC7A35T-2FGG484I, U9 SIT9121AI-2BF-XXS156.250000G

Commit message: Under 100 unrouted
Parts:
- added J25: PMOD_HOST, azonenberg_pcb:CONN_HEADER_2.54MM_2x6_RA_PMOD_HOST, symbol special-azonenberg:PMOD_HOST
Connections:
- net 3V3: now also J25.12 (3V3), J25.6 (3V3)
- net FPGA_UART_CTS_N: now also J6.6 (P6); no longer J6.2 (P2)
- net FPGA_UART_RTS_N: now also J6.2 (P2), U4.A21 (IO_L21N_T3_DQS_16); no longer J6.6 (P6), U4.A20 (IO_L16N_T2_16)
- net FPGA_UART_RX: now also J6.4 (P4), U4.A20 (IO_L16N_T2_16); no longer J6.5 (P5), U4.A21 (IO_L21N_T3_DQS_16)
- net FPGA_UART_TX: now also J6.5 (P5); no longer J6.4 (P4)
- net GND: now also J25.11 (GND), J25.5 (GND)
- net FPGA_PMOD_DQ4: now reaches U4.A13 (IO_L10P_T1_16)
- net FPGA_PMOD_DQ4: now also J25.7 (D4)
- net FPGA_PMOD_DQ5: now reaches U4.A14 (IO_L10N_T1_16)
- net FPGA_PMOD_DQ5: now also J25.8 (D5)
- net FPGA_PMOD_DQ6: now reaches U4.A15 (IO_L9P_T1_DQS_16)
- net FPGA_PMOD_DQ6: now also J25.9 (D6)
- net FPGA_PMOD_DQ7: now reaches U4.A16 (IO_L9N_T1_DQS_16)
- net FPGA_PMOD_DQ7: now also J25.10 (D7)
- net FPGA_PMOD_DQ0: now reaches U4.B13 (IO_L8N_T1_16)
- net FPGA_PMOD_DQ0: now also J25.1 (D0)
- net FPGA_PMOD_DQ2: now reaches U4.B15 (IO_L7P_T1_16)
- net FPGA_PMOD_DQ2: now also J25.3 (D2)
- net FPGA_PMOD_DQ3: now reaches U4.B16 (IO_L7N_T1_16)
- net FPGA_PMOD_DQ3: now also J25.4 (D3)
- net FPGA_PMOD_DQ1: now reaches U4.C14 (IO_L3P_T0_DQS_16)
- net FPGA_PMOD_DQ1: now also J25.2 (D1)
- no-connect marks 199 -> 191

Commit message: Continued layout
Connections:
- net LED_CTRL: now also U4.B21 (IO_L21P_T3_DQS_16); no longer U4.F21 (IO_25_16)
- net at R54.2: now also U4.R2 (IO_L3N_T0_DQS_34); no longer U4.T1 (IO_L1P_T0_34)
- net at R56.2: now also U4.U1 (IO_L1N_T0_34); no longer U4.U2 (IO_L2P_T0_34)
- net at R55.2: now also U4.T1 (IO_L1P_T0_34); no longer U4.U1 (IO_L1N_T0_34)
Other:
- moved on the sheet: R54, R55, R56
Changed lines of the file:
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@@
 	(title_block
 		(title "Oscilloscope Demo Board")
-		(date "2026-08-11")
+		(date "2026-08-12")
 		(rev "0.1")
 		(company "Antikernel Labs")
@@
 	)
 	(no_connect
+		(at 123.19 144.78)
+	)
+	(no_connect
 		(at 262.89 119.38)
 	)
@@
 	)
 	(no_connect
-		(at 123.19 124.46)
-	)
-	(no_connect
 		(at 43.18 127)
 	)
@@
 	)
 	(no_connect
-		(at 191.77 35.56)
-	)
-	(no_connect
 		(at 262.89 116.84)
 	)
@@
 	)
 	(no_connect
+		(at 191.77 27.94)
+	)
+	(no_connect
 		(at 123.19 45.72)
 	)
@@
 	(wire
 		(pts
-			(xy 186.69 27.94) (xy 191.77 27.94)
+			(xy 186.69 35.56) (xy 191.77 35.56)
 		)
 		(stroke
@@
 	)
 	(label "COAX_1"
-		(at 179.07 22.86 180)
+		(at 179.07 35.56 180)
 		(effects
 			(font
@@
 	)
 	(label "COAX_2"
-		(at 179.07 25.4 180)
+		(at 179.07 22.86 180)
 		(effects
 			(font
@@
 	)
 	(label "COAX_3"
-		(at 179.07 27.94 180)
+		(at 179.07 25.4 180)
 		(effects
 			(font
@@
 	)
 	(label "LED_CTRL"
-		(at 123.19 144.78 180)
+		(at 123.19 124.46 180)
 		(effects
 			(font
@@
 	(symbol
 		(lib_id "device:R")
-		(at 182.88 22.86 90)
+		(at 182.88 35.56 90)
 		(unit 1)
 		(exclude_from_sim no)
@@
 		(dnp no)
 		(property "Reference" "R54"
-			(at 187.96 21.59 90)
+			(at 187.96 34.29 90)
 			(effects
 				(font
@@
 		)
 		(property "Value" "33"
-			(at 182.88 22.86 90)
+			(at 182.88 35.56 90)
 			(effects
 				(font
@@
 		)
 		(property "Footprint" "azonenberg_pcb:EIA_0402_RES_NOSILK"
-			(at 182.88 24.638 90)
+			(at 182.88 37.338 90)
 			(effects
 				(font
@@
 		)
 		(property "Datasheet" ""
-			(at 182.88 22.86 0)
+			(at 182.88 35.56 0)
 			(effects
 				(font
@@
 		)
 		(property "Description" "Resistor"
-			(at 182.88 22.86 0)
+			(at 182.88 35.56 0)
 			(effects
 				(font
@@
 	(symbol
 		(lib_id "device:R")
-		(at 182.88 27.94 90)
+		(at 182.88 25.4 90)
 		(unit 1)
 		(exclude_from_sim no)
@@
 		(dnp no)
 		(property "Reference" "R56"
-			(at 187.96 26.67 90)
+			(at 187.96 24.13 90)
 			(effects
 				(font
@@
 		)
 		(property "Value" "33"
-			(at 182.88 27.94 90)
+			(at 182.88 25.4 90)
 			(effects
 				(font
@@
 		)
 		(property "Footprint" "azonenberg_pcb:EIA_0402_RES_NOSILK"
-			(at 182.88 29.718 90)
+			(at 182.88 27.178 90)
 			(effects
 				(font
@@
 		)
 		(property "Datasheet" ""
-			(at 182.88 27.94 0)
+			(at 182.88 25.4 0)
 			(effects
 				(font
@@
 		)
 		(property "Description" "Resistor"
-			(at 182.88 27.94 0)
+			(at 182.88 25.4 0)
 			(effects
 				(font
@@
 	(symbol
 		(lib_id "device:R")
-		(at 182.88 25.4 90)
+		(at 182.88 22.86 90)
 		(unit 1)
 		(exclude_from_sim no)
@@
 		(dnp no)
 		(property "Reference" "R55"
-			(at 187.96 24.13 90)
+			(at 187.96 21.59 90)
 			(effects
 				(font
@@
 		)
 		(property "Value" "33"
-			(at 182.88 25.4 90)
+			(at 182.88 22.86 90)
 			(effects
 				(font
@@
 		)
 		(property "Footprint" "azonenberg_pcb:EIA_0402_RES_NOSILK"
-			(at 182.88 27.178 90)
+			(at 182.88 24.638 90)
 			(effects
 				(font
@@
 		)
 		(property "Datasheet" ""
-			(at 182.88 25.4 0)
+			(at 182.88 22.86 0)
 			(effects
 				(font
@@
 		)
 		(property "Description" "Resistor"
-			(at 182.88 25.4 0)
+			(at 182.88 22.86 0)
 			(effects
 				(font

Commit message: Finished initial routing of demo board but might still add more features
Parts:
- added J26, J27: TESTCLIP, azonenberg_pcb:TESTPOINT_SMT_KEYSTONE_5016, symbol conn:CONN_01X01
Connections:
- net CLIP_1: now also U4.G20 (IO_L8N_T1_AD10N_15); no longer U4.H14 (IO_L3N_T0_DQS_AD1N_15)
- net CLIP_2: now also U4.H22 (IO_L7N_T1_AD2N_15); no longer U4.G17 (IO_L4P_T0_AD9P_15)
- net CLIP_3: now also U4.J21 (IO_L11N_T1_SRCC_15); no longer U4.G18 (IO_L4N_T0_AD9N_15)
- net CLIP_4: now also U4.J22 (IO_L7P_T1_AD2P_15); no longer U4.J15 (IO_L5P_T0_AD9P_15)
- net GND: now also J26.1 (P1), J27.1 (P1)
Changed lines of the file:
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@@
 	(title_block
 		(title "Oscilloscope Demo Board")
-		(date "2026-08-12")
+		(date "2026-08-13")
 		(rev "0.1")
 		(company "Antikernel Labs")
@@
 	)
 	(no_connect
-		(at 43.18 76.2)
-	)
-	(no_connect
 		(at 262.89 76.2)
 	)
@@
 	)
 	(no_connect
+		(at 43.18 38.1)
+	)
+	(no_connect
 		(at 335.28 27.94)
 	)
@@
 	)
 	(no_connect
+		(at 43.18 35.56)
+	)
+	(no_connect
 		(at 191.77 96.52)
 	)
@@
 	)
 	(no_connect
-		(at 43.18 60.96)
-	)
-	(no_connect
 		(at 191.77 104.14)
 	)
@@
 	)
 	(no_connect
+		(at 43.18 43.18)
+	)
+	(no_connect
 		(at 262.89 127)
 	)
@@
 	)
 	(no_connect
-		(at 43.18 53.34)
-	)
-	(no_connect
 		(at 43.18 99.06)
 	)
@@
 	)
 	(no_connect
-		(at 43.18 55.88)
-	)
-	(no_connect
 		(at 43.18 139.7)
 	)
@@
 	)
 	(no_connect
+		(at 43.18 40.64)
+	)
+	(no_connect
 		(at 262.89 38.1)
 	)
@@
 	)
 	(label "CLIP_3"
-		(at 43.18 40.64 180)
+		(at 43.18 76.2 180)
 		(effects
 			(font
@@
 		)
 	)
+	(label "GND"
+		(at 106.68 189.23 180)
+		(effects
+			(font
+				(size 1.27 1.27)
+			)
+			(justify right bottom)
+		)
+	)
 	(label "COAX_3"
 		(at 179.07 25.4 180)
@@
 		)
 	)
+	(label "GND"
+		(at 106.68 195.58 180)
+		(effects
+			(font
+				(size 1.27 1.27)
+			)
+			(justify right bottom)
+		)
+	)
 	(label "FPGA_LED1"
 		(at 265.43 256.54 180)
@@
 	)
 	(label "CLIP_2"
-		(at 43.18 38.1 180)
+		(at 43.18 55.88 180)
 		(effects
 			(font
@@
 	)
 	(label "CLIP_1"
-		(at 43.18 35.56 180)
+		(at 43.18 60.96 180)
 		(effects
 			(font
@@
 	)
 	(label "CLIP_4"
-		(at 43.18 43.18 180)
+		(at 43.18 53.34 180)
 		(effects
 			(font
@@
 	)
 	(symbol
+		(lib_id "conn:CONN_01X01")
+		(at 111.76 195.58 0)
+		(unit 1)
+		(exclude_from_sim no)
+		(in_bom yes)
+		(on_board yes)
+		(dnp no)
+		(fields_autoplaced yes)
+		(property "Reference" "J27"
+			(at 113.665 194.3678 0)
+			(effects
+				(font
+					(size 1.27 1.27)
+				)
+				(justify left)
+			)
+		)
+		(property "Value" "TESTCLIP"
+			(at 113.665 196.7921 0)
+			(effects
+				(font
+					(size 1.27 1.27)
+				)
+				(justify left)
+			)
+		)
+		(property "Footprint" "azonenberg_pcb:TESTPOINT_SMT_KEYSTONE_5016"
+			(at 111.76 195.58 0)
+			(effects
+				(font
+					(size 1.27 1.27)
+				)
+				(hide yes)
+			)
+		)
+		(property "Datasheet" ""
+			(at 111.76 195.58 0)
+			(effects
+				(font
+					(size 1.27 1.27)
+				)
+				(hide yes)
+			)
+		)
+		(property "Description" "Connector, single row, 01x01, pin header"
+			(at 111.76 195.58 0)
+			(effects
+				(font
+					(size 1.27 1.27)
+				)
+				(hide yes)
+			)
+		)
+		(pin "1"
+		)
+		(instances
+			(project "demo-board"
+				(path "/aa2d82c6-7ba7-4266-9b47-ed3339e6c556/a5c6d6a0-0eb9-4128-8a96-febfa5d4e510"
+					(reference "J27")
+					(unit 1)
+				)
+			)
+		)
+	)
+	(symbol
 		(lib_id "device:C")
 		(at 85.09 273.05 0)
@@
 					(unit 1)
 				)
+			)
+		)
+	)
+	(symbol
+		(lib_id "conn:CONN_01X01")
+		(at 111.76 189.23 0)
+		(unit 1)
+		(exclude_from_sim no)
+		(in_bom yes)
+		(on_board yes)
+		(dnp no)
+		(fields_autoplaced yes)
+		(property "Reference" "J26"
+			(at 113.665 188.0178 0)
+			(effects
+				(font
+					(size 1.27 1.27)
+				)
+				(justify left)
+			)
+		)
+		(property "Value" "TESTCLIP"
+			(at 113.665 190.4421 0)
+			(effects
+				(font
+					(size 1.27 1.27)
+				)
+				(justify left)
+			)
+		)
+		(property "Footprint" "azonenberg_pcb:TESTPOINT_SMT_KEYSTONE_5016"
+			(at 111.76 189.23 0)
+			(effects
+				(font
+					(size 1.27 1.27)
+				)
+				(hide yes)
+			)
+		)
+		(property "Datasheet" ""
+			(at 111.76 189.23 0)
+			(effects
+				(font
+					(size 1.27 1.27)
+				)
+				(hide yes)
+			)
+		)
+		(property "Description" "Connector, single row, 01x01, pin header"
+			(at 111.76 189.23 0)
+			(effects
+				(font
+					(size 1.27 1.27)
+				)
+				(hide yes)
+			)
+		)
+		(pin "1"
+		)
+		(instances
+			(project "demo-board"
+				(path "/aa2d82c6-7ba7-4266-9b47-ed3339e6c556/a5c6d6a0-0eb9-4128-8a96-febfa5d4e510"
+					(reference "J26")
+					(unit 1)
+				)
