File: oscilloscope-probing/lab/boards/demo-board/testsignals.kicad_sch (KiCad schematic)
At the start: 56 parts, among them J10 SMA-J-P-H-ST-EM1, J11 TESTCLIP, J12 TESTCLIP, J13 TESTCLIP, J15 TESTCLIP, J16 SMA-J-P-H-ST-EM1, J17 SMA-J-P-H-ST-EM1, J18 SMA-J-P-H-ST-EM1, J19 SMA-J-P-H-ST-EM1, J20 SMA-J-P-H-ST-EM1, J21 SMA-J-P-H-ST-EM1, J22 SMA-J-P-H-ST-EM1, J23 SMA-J-P-H-ST-EM1, J25 PMOD_HOST, J26 TESTCLIP, J27 TESTCLIP, J6 CONN_01X06, J7 SMA-J-P-H-ST-EM1, J8 SMA-J-P-H-ST-EM1, J9 SMA-J-P-H-ST-EM1, U10 19-C47/RSGHBHC-5V01/2T, U11 19-C47/RSGHBHC-5V01/2T, U12 19-C47/RSGHBHC-5V01/2T, U13 19-C47/RSGHBHC-5V01/2T, U26 74LVC1T45, U4 XC7A35T-2FGG484I, U9 SIT9121AI-2BF-XXS156.250000G

Commit message: Various updates made during design review
Parts:
- added J30: TESTCLIP, azonenberg_pcb:TESTPOINT_SMT_KEYSTONE_5016, symbol conn:CONN_01X01
Connections:
- net GND: now also J30.1 (P1)
Changed lines of the file:
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@@
 		)
 	)
+	(label "GND"
+		(at 106.68 201.93 180)
+		(effects
+			(font
+				(size 1.27 1.27)
+			)
+			(justify right bottom)
+		)
+	)
 	(label "GTP_REF_P"
 		(at 335.28 81.28 180)
@@
 				)
 			)
+		)
+	)
+	(symbol
+		(lib_id "conn:CONN_01X01")
+		(at 111.76 201.93 0)
+		(unit 1)
+		(exclude_from_sim no)
+		(in_bom yes)
+		(on_board yes)
+		(dnp no)
+		(fields_autoplaced yes)
+		(property "Reference" "J30"
+			(at 113.665 200.7178 0)
+			(effects
+				(font
+					(size 1.27 1.27)
+				)
+				(justify left)
+			)
+		)
+		(property "Value" "TESTCLIP"
+			(at 113.665 203.1421 0)
+			(effects
+				(font
+					(size 1.27 1.27)
+				)
+				(justify left)
+			)
+		)
+		(property "Footprint" "azonenberg_pcb:TESTPOINT_SMT_KEYSTONE_5016"
+			(at 111.76 201.93 0)
+			(effects
+				(font
+					(size 1.27 1.27)
+				)
+				(hide yes)
+			)
+		)
+		(property "Datasheet" ""
+			(at 111.76 201.93 0)
+			(effects
+				(font
+					(size 1.27 1.27)
+				)
+				(hide yes)
+			)
+		)
+		(property "Description" "Connector, single row, 01x01, pin header"
+			(at 111.76 201.93 0)
+			(effects
+				(font
+					(size 1.27 1.27)
+				)
+				(hide yes)
+			)
+		)
+		(pin "1"
+		)
+		(instances
+			(project "demo-board"
+				(path "/aa2d82c6-7ba7-4266-9b47-ed3339e6c556/a5c6d6a0-0eb9-4128-8a96-febfa5d4e510"
+					(reference "J30")
+					(unit 1)
+				)
+			)
