File: oscilloscope-probing/lab/boards/demo-board/mcu.kicad_sch (KiCad schematic)
At the start: 75 parts, among them J24 PMOD_HOST, J4 CORTEX_DEBUG_ETM, SW3 SWITCH, SW4 SWITCH, SW5 SWITCH, SW6 SWITCH, SW7 SWITCH, U4 XC7A35T-2FGG484I, U5 STM32H750XBH6, U6 ECS-1612MV-250-CN, U7 ECS-1612MV-250-CN, U8 S25FL064LABMFI013

Commit message: Continued layout
Connections:
- net MCU_PMOD_DQ0: now also U5.H2 (PI13); no longer U5.U4 (PC5)
- net MCU_PMOD_DQ1: now also U5.G3 (PF1); no longer U5.T5 (PB1)
- net MCU_PMOD_DQ2: now also U5.E2 (PI9); no longer U5.U2 (PA3)
- net MCU_PMOD_DQ3: now also U5.E3 (PC13); no longer U5.T4 (PC4)
- net MCU_PMOD_DQ4: now also U5.H1 (PI12); no longer U5.R3 (PA6)
- net MCU_PMOD_DQ5: now also U5.G1 (PF2); no longer U5.N2 (PH2)
- net MCU_PMOD_DQ6: now also U5.F3 (PI10); no longer U5.P2 (PH3)
- net MCU_PMOD_DQ7: now also U5.H3 (PI14); no longer U5.P3 (PH4)
- net MCU_TRIG: now also U5.D6 (PG15); no longer U5.C1 (PC15)
Other:
- moved on the sheet: TP12
Changed lines of the file:
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@@
 	(title_block
 		(title "Oscilloscope Demo Board")
-		(date "2026-08-11")
+		(date "2026-08-12")
 		(rev "0.1")
 		(company "Antikernel Labs")
@@
 	)
 	(no_connect
+		(at 35.56 73.66)
+	)
+	(no_connect
 		(at 35.56 54.61)
 	)
@@
 	)
 	(no_connect
-		(at 35.56 156.21)
-	)
-	(no_connect
 		(at 35.56 151.13)
 	)
@@
 	)
 	(no_connect
+		(at 35.56 135.89)
+	)
+	(no_connect
 		(at 158.75 36.83)
 	)
@@
 	)
 	(no_connect
-		(at 107.95 109.22)
-	)
-	(no_connect
-		(at 107.95 195.58)
+		(at 35.56 161.29)
 	)
 	(no_connect
@@
 	)
 	(no_connect
-		(at 107.95 200.66)
-	)
-	(no_connect
 		(at 35.56 146.05)
 	)
 	(no_connect
-		(at 107.95 29.21)
-	)
-	(no_connect
 		(at 107.95 49.53)
 	)
@@
 	)
 	(no_connect
-		(at 107.95 205.74)
-	)
-	(no_connect
 		(at 107.95 99.06)
 	)
@@
 	)
 	(no_connect
+		(at 35.56 158.75)
+	)
+	(no_connect
 		(at 35.56 96.52)
 	)
@@
 	)
 	(no_connect
-		(at 107.95 198.12)
-	)
-	(no_connect
 		(at 107.95 247.65)
 	)
@@
 	)
 	(no_connect
+		(at 35.56 39.37)
+	)
+	(no_connect
 		(at 35.56 52.07)
 	)
@@
 	)
 	(no_connect
-		(at 107.95 26.67)
+		(at 107.95 133.35)
 	)
 	(no_connect
-		(at 107.95 133.35)
+		(at 35.56 31.75)
 	)
 	(no_connect
@@
 	)
 	(no_connect
+		(at 35.56 133.35)
+	)
+	(no_connect
+		(at 107.95 125.73)
+	)
+	(no_connect
 		(at 250.19 182.88)
 	)
@@
 	)
 	(no_connect
+		(at 107.95 198.12)
+	)
+	(no_connect
 		(at 250.19 185.42)
 	)
@@
 	)
 	(no_connect
-		(at 107.95 203.2)
-	)
-	(no_connect
-		(at 35.56 158.75)
-	)
-	(no_connect
 		(at 35.56 99.06)
 	)
@@
 	)
 	(no_connect
-		(at 107.95 59.69)
+		(at 107.95 123.19)
 	)
 	(no_connect
-		(at 107.95 193.04)
+		(at 107.95 59.69)
 	)
 	(no_connect
@@
 	)
 	(no_connect
+		(at 107.95 128.27)
+	)
+	(no_connect
 		(at 347.98 26.67)
 	)
@@
 	(wire
 		(pts
-			(xy 24.13 161.29) (xy 35.56 161.29)
+			(xy 96.52 109.22) (xy 107.95 109.22)
 		)
 		(stroke
@@
 	)
 	(label "MCU_PMOD_DQ5"
-		(at 107.95 123.19 180)
+		(at 107.95 29.21 180)
 		(effects
 			(font
@@
 	)
 	(label "MCU_PMOD_DQ7"
-		(at 107.95 128.27 180)
+		(at 107.95 205.74 180)
 		(effects
 			(font
@@
 	)
 	(label "MCU_PMOD_DQ0"
-		(at 35.56 135.89 180)
+		(at 107.95 203.2 180)
 		(effects
 			(font
@@
 	)
 	(label "MCU_PMOD_DQ2"
-		(at 35.56 31.75 180)
+		(at 107.95 193.04 180)
 		(effects
 			(font
@@
 	)
 	(label "MCU_PMOD_DQ4"
-		(at 35.56 39.37 180)
+		(at 107.95 200.66 180)
 		(effects
 			(font
@@
 	)
 	(label "MCU_PMOD_DQ6"
-		(at 107.95 125.73 180)
+		(at 107.95 195.58 180)
 		(effects
 			(font
@@
 	)
 	(label "MCU_TRIG"
-		(at 24.13 161.29 0)
+		(at 96.52 109.22 0)
 		(effects
 			(font
@@
 	)
 	(label "MCU_PMOD_DQ1"
-		(at 35.56 73.66 180)
+		(at 107.95 26.67 180)
 		(effects
 			(font
@@
 	)
 	(label "MCU_PMOD_DQ3"
-		(at 35.56 133.35 180)
+		(at 35.56 156.21 180)
 		(effects
 			(font
@@
 	(symbol
 		(lib_id "conn:CONN_01X01")
-		(at 19.05 161.29 0)
+		(at 91.44 109.22 0)
 		(mirror y)
 		(unit 1)
@@
 		(dnp no)
 		(property "Reference" "TP12"
-			(at 21.59 163.83 0)
+			(at 93.98 111.76 0)
 			(effects
 				(font
@@
 		)
 		(property "Value" "TESTCLIP"
-			(at 21.59 166.2543 0)
+			(at 93.98 114.1843 0)
 			(effects
 				(font
@@
 		)
 		(property "Footprint" "azonenberg_pcb:TESTPOINT_SMT_KEYSTONE_5016"
-			(at 19.05 161.29 0)
+			(at 91.44 109.22 0)
 			(effects
 				(font
@@
 		)
 		(property "Datasheet" ""
-			(at 19.05 161.29 0)
+			(at 91.44 109.22 0)
 			(effects
 				(font
@@
 		)
 		(property "Description" "Connector, single row, 01x01, pin header"
-			(at 19.05 161.29 0)
+			(at 91.44 109.22 0)
 			(effects
 				(font

Commit message: Finished initial routing of demo board but might still add more features
Connections:
- net DPY_BS: now also U5.B16 (PH15); no longer U5.A16 (PI0)
- net DPY_BUSY_N: now also U5.A16 (PI0); no longer U5.B16 (PH15)
- net DPY_DC: now also U5.A15 (PI1); no longer U5.B15 (PI2)
- net DPY_RST_N: now also U5.B15 (PI2); no longer U5.A15 (PI1)
- net FMC_A22: now also U4.P15 (IO_L22P_T3_A05_D21_14); no longer U4.U20 (IO_L11P_T1_SRCC_14)
- net FMC_AD2: now also U4.U20 (IO_L11P_T1_SRCC_14); no longer U4.T18 (IO_L20N_T3_A07_D23_14)
- net FMC_AD8: now also U4.R18 (IO_L20P_T3_A08_D24_14); no longer U4.P15 (IO_L22P_T3_A05_D21_14)
- net FMC_NE3: now also U4.T18 (IO_L20N_T3_A07_D23_14); no longer U4.R18 (IO_L20P_T3_A08_D24_14)
Changed lines of the file:
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@@
 	(title_block
 		(title "Oscilloscope Demo Board")
-		(date "2026-08-12")
+		(date "2026-08-13")
 		(rev "0.1")
 		(company "Antikernel Labs")
@@
 	)
 	(label "DPY_BUSY_N"
-		(at 107.95 156.21 180)
+		(at 107.95 170.18 180)
 		(effects
 			(font
@@
 	)
 	(label "FMC_A22"
-		(at 347.98 80.01 180)
+		(at 347.98 135.89 180)
 		(effects
 			(font
@@
 	)
 	(label "DPY_RST_N"
-		(at 107.95 172.72 180)
+		(at 107.95 175.26 180)
 		(effects
 			(font
@@
 	)
 	(label "DPY_BS"
-		(at 107.95 170.18 180)
+		(at 107.95 156.21 180)
 		(effects
 			(font
@@
 	)
 	(label "FMC_AD2"
-		(at 347.98 128.27 180)
+		(at 347.98 80.01 180)
 		(effects
 			(font
@@
 	)
 	(label "FMC_NE3"
-		(at 347.98 125.73 180)
+		(at 347.98 128.27 180)
 		(effects
 			(font
@@
 	)
 	(label "DPY_DC"
-		(at 107.95 175.26 180)
+		(at 107.95 172.72 180)
 		(effects
 			(font
@@
 	)
 	(label "FMC_AD8"
-		(at 347.98 135.89 180)
+		(at 347.98 125.73 180)
 		(effects
 			(font

Commit message: Demo board is done ish awaiting final design review
Parts:
- added J28, J29: SMA-J-P-H-ST-EM1, azonenberg_pcb:CONN_SMA_EDGE_SAMTEC_SMA_J_P_H_ST_EM1_NOPASTE, symbol conn:CONN_COAXIAL
- added R67, R68: 127, azonenberg_pcb:EIA_0402_RES_NOSILK, symbol device:R
Connections:
- net GND: now also J28.2 (Ext), J29.2 (Ext)
- net PAM3_TX_P: now reaches U4.P19 (IO_L5P_T0_D06_14)
- net PAM3_TX_P: now also R67.1
- net PAM3_TX_N: now reaches U4.R19 (IO_L5N_T0_D07_14)
- net PAM3_TX_N: now also R68.1
- new net: J28.1 (In), R67.2
- new net: J29.1 (In), R68.2
- no-connect marks 110 -> 108
